File: graphic.brd (EAGLE design)
At the start: 109 x 29.5 mm, 72 parts, among them IC1 NE5532D, IC2 NE5532D, IC3 NE5532D, IC4 NE5532D, IC5 NE5532D, U2 THONKICONNNEW, U3 THONKICONNNEW

Commit message: Simple version PCB complete and routed
Parts:
- removed D1, D2: PMEG2010AEB, diode:SOD523
- removed L1, L2: (no value), wuerth-elektronik:0603
- removed U2, U3: THONKICONNNEW, MusicThingModular:WQP-PJ301M-12_JACK
- added C28, C29, C30: 100n, we-rcl:C0805
- added D3, D4: 5819, diode:SOD123
- added INPUT, OUTPUT: THONKICONNNEW, MusicThingModular:WQP-PJ301M-12_JACK
- C12, C13, C4, C6, C9: device rcl:C0402 -> we-rcl:C0805
- moved C4 115.7 mm to (13.0, 15.9), turned to 90 degrees
- moved C12 99.7 mm to (27.9, 9.84)
- moved R6 93.2 mm to (25.4, 22.9), turned to 90 degrees
- moved C22 93.0 mm to (25.4, 21.0), turned to 90 degrees
- moved C9 92.1 mm to (27.9, 16.8)
- moved R9 87.6 mm to (38.1, 19.1), turned to 90 degrees
- moved IC3 81.7 mm to (45.7, 13.3)
- moved R8 75.8 mm to (38.1, 22.9), turned to 90 degrees
- moved C20 74.2 mm to (85.7, 24.8), turned to 90 degrees
- moved C23 73.9 mm to (38.1, 21.0), turned to 90 degrees
- moved R10 69.2 mm to (49.5, 22.9), turned to 90 degrees
- moved R1 68.3 mm to (3.81, 13.3), turned to 180 degrees
- moved C24 67.6 mm to (49.5, 21.0), turned to 90 degrees
- moved R11 66.1 mm to (49.5, 19.1), turned to 90 degrees
- moved R25 65.7 mm to (7.62, 21.0), turned to 90 degrees
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Connections:
- removed net N$22: D1.C, L1.2
- removed net N$44: D2.A, L2.2
- removed net V+: IC1.8, IC2.8, IC3.8, IC4.8, IC5.8
- removed net V-: IC1.4, IC2.4, IC3.4, IC4.4, IC5.4
- removed net VCC: C1.1, C13.1, C4.1, C9.1
- removed net VEE: C12.2, C2.2, C6.2
- net +12V: now also C1.1, C13.2, C29.2, C4.2, C9.2, D3.C, IC1.8, IC2.8, IC3.8, IC4.8, IC5.8; no longer L1.1, R18.2, R19.2, R20.2, R21.2, R22.2, R23.2, R24.2
- net +_INLET: now also D3.A, R18.2, R19.2, R20.2, R21.2, R22.2, R23.2, R24.2; no longer D1.A
- net -12V: now also C12.1, C2.1, C28.1, C30.1, C6.1, D4.A, IC1.4, IC2.4, IC3.4, IC4.4, IC5.4; no longer L2.1
- net -_INLET: now also D4.C; no longer D2.C
- net GND: now also C12.2, C13.1, C2.2, C28.2, C29.1, C30.2, C4.1, C6.2, C9.1, INPUT.P$3_SLEEVE, OUTPUT.P$3_SLEEVE, R11.2, R15.2, R17.2, R7.2; no longer C12.1, C13.2, C2.1, C4.2, C6.1, C9.2, R11.1, R15.1, R17.1, R7.1, U2.P$3_SLEEVE, U3.P$3_SLEEVE
- net N$11: now also C17.1; no longer C17.2
- net N$12: now also C15.1, C16.1; no longer C15.2, C16.2
- net N$14: now also C10.1, C8.1; no longer C10.2, C8.2
- net N$16: now also C23.2, IC3.3; no longer C23.1, IC3.2
- net N$17: now also C21.1, C3.2, C7.2; no longer C21.2, C3.1, C7.1
- net N$18: now also C10.2, C8.2, R6.2; no longer C10.1, C8.1, R6.1
- net N$19: now also C18.1, C19.1; no longer C18.2, C19.2
- net N$2: now also INPUT.P$1_TIP; no longer U2.P$1_TIP
- net N$21: now also IC3.2; no longer IC3.3
- net N$23: now also C20.1; no longer C20.2
- net N$24: now also IC3.5, R11.1; no longer IC3.6, R11.2
- net N$25: now also C21.2, IC2.3; no longer C21.1, IC2.2
- net N$26: now also IC2.2; no longer IC2.3
- net N$27: now also IC3.6, R10.1; no longer IC3.5, R10.2
- net N$28: now also IC2.5, R7.1; no longer IC2.6, R7.2
- net N$29: now also IC2.6, R6.1; no longer IC2.5, R6.2
- net N$3: now also R1.1; no longer R1.2
- net N$30: now also C11.2, C14.2, C23.1; no longer C11.1, C14.1, C23.2
- net N$31: now also C15.2, C16.2, R10.2; no longer C15.1, C16.1, R10.1
- net N$32: now also C25.2, IC4.3; no longer C25.1, IC4.2
- net N$33: now also IC4.2; no longer IC4.3
- net N$34: now also IC4.5, R15.1; no longer IC4.6, R15.2
- net N$35: now also IC4.6, R14.1; no longer IC4.5, R14.2
- net N$36: now also C17.2, C25.1; no longer C17.1, C25.2
- net N$37: now also C18.2, C19.2, R14.2; no longer C18.1, C19.1, R14.1
- net N$38: now also IC5.5, R17.1; no longer IC5.6, R17.2
- net N$39: now also IC5.6, R16.1; no longer IC5.5, R16.2
- net N$4: now also C11.1, C14.1; no longer C11.2, C14.2
- net N$40: now also C20.2, R16.2; no longer C20.1, R16.1
- net N$45: now also R1.2, R26.1; no longer R1.1, R26.2
- net N$5: now also R3.2; no longer R3.1
- net N$6: now also OUTPUT.P$1_TIP, R3.1; no longer R3.2, U3.P$1_TIP
- net N$8: now also C3.1, C7.1; no longer C3.2, C7.2
- net N$9: now also R26.2; no longer R26.1
Routing:
- net N$6: track 0.00 -> 124.5 mm, vias 0 -> 1
- net N$1: track 106.7 -> 0.00 mm
- net +_INLET: track 0.00 -> 105.7 mm
- net N$3: track 0.00 -> 105.0 mm
- net +12V: track 0.00 -> 98.0 mm
- net N$7: track 0.00 -> 97.7 mm, vias 0 -> 1
- net -12V: track 0.00 -> 94.9 mm
- net N$16: track 0.00 -> 21.0 mm, vias 0 -> 2
- net N$32: track 0.00 -> 20.1 mm, vias 0 -> 2
- net N$25: track 0.00 -> 19.1 mm, vias 0 -> 2
- net N$2: track 0.00 -> 18.4 mm
- net N$8: track 0.00 -> 18.0 mm
- net N$21: track 0.00 -> 17.2 mm, vias 0 -> 2
- net N$33: track 0.00 -> 17.2 mm, vias 0 -> 2
- net GND: track 0.00 -> 16.8 mm
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- added copper zone on layer 1, net GND
- added copper zone on layer 16, net GND
Other:
- board text added: "Graphic EQ Designed in Herne HIll, London, by Tom Whitwell January 2017 Proto 1"
- board text added: "n$3 = CUT n$7 = boost 75ml placement grid 12.5mil routing grid"
