File: graphic_panel.brd (EAGLE design)
At the start: 128.5 x 30 mm, 3 parts

Commit message: re route and redesign panel
Parts:
- added E$1, E$2, E$3, E$4, E$5, E$6, E$7: (no value), MusicThingModular:20MM_SLOT
Other:
- outline, holes or cut-outs redrawn
- board text added: "Graphic EQ Designed in Herne HIll, London, by Tom Whitwell February 2017 Proto 2"
- board text added: "MUSIC THING MODULAR"
- board text removed: "Graphic EQ Designed in Herne HIll, London, by Tom Whitwell January 2017 Proto 1"

Commit message: Updated illuminated fader outline
Changed lines of the file:
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@@
 <text x="24.0375" y="1.2025" size="1.016" layer="21">Graphic EQ Designed in Herne HIll, London, by Tom Whitwell February 2017 Proto 2</text>
 <rectangle x1="0" y1="0" x2="12" y2="30" layer="29"/>
-<rectangle x1="119" y1="0" x2="128.5" y2="30" layer="29"/>
+<rectangle x1="116" y1="0" x2="128.5" y2="30" layer="29"/>
 <wire x1="0" y1="0" x2="0" y2="30" width="0" layer="20"/>
 <text x="125.5" y="2.5" size="1.778" layer="22" rot="SMR270" align="center-right">GRAPHIC</text>
