File: graphic.sch (EAGLE design)
At the start: 81 parts, among them IC1 NE5532D, IC2 NE5532D, IC3 NE5532D, IC4 NE5532D, IC5 NE5532D

Commit message: Tweaks for Rev 1 boards: improve ground plane clearance, move one resistor, move Kills Fascists arwork, small changes to get ground plane to work
Parts:
- added FID1, FID2: FIDUCIAL1X2.5, SparkFun-Aesthetics:FIDUCIAL1X2.5
Changed lines of the file:
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@@
 <?xml version="1.0" encoding="utf-8"?>
 <!DOCTYPE eagle SYSTEM "eagle.dtd">
-<eagle version="7.2.0">
+<eagle version="7.7.0">
 <drawing>
 <settings>
@@
 <part name="C37" library="we-rcl" deviceset="CAPACITOR" device="-0805" value="NP"/>
 <part name="C38" library="we-rcl" deviceset="CAPACITOR" device="-0805" value="NP"/>
+<part name="FID1" library="SparkFun-Aesthetics" deviceset="FIDUCIAL" device="1X2.5"/>
+<part name="FID2" library="SparkFun-Aesthetics" deviceset="FIDUCIAL" device="1X2.5"/>
 </parts>
 <sheets>
@@
 <instance part="C37" gate="C" x="284.48" y="121.92" rot="R270"/>
 <instance part="C38" gate="C" x="292.1" y="121.92" rot="R270"/>
+<instance part="FID1" gate="G$1" x="20.32" y="33.02"/>
+<instance part="FID2" gate="G$1" x="27.94" y="33.02"/>
 </instances>
 <busses>
