File: graphic_stereo.sch (EAGLE design)
At the start: 81 parts, among them IC1 NE5532D, IC2 NE5532D, IC3 NE5532D, IC4 NE5532D, IC5 NE5532D

Commit message: Revert "Tweaks for Rev 1 boards: improve ground plane clearance, move one resistor, move Kills Fascists arwork, small changes to get ground plane to work"
This reverts commit c469b6aed1205b33f2cf1fbab66cd5b8357eaae7.
Parts:
- removed C31, C32, C33, C34, C35, C36, C37, C38: NP, we-rcl:CAPACITOR-0805
- added IC6: NE5532D, linear:NE5532D
- added L_OUT, R_OUT: THONKICONNNEW, MusicThingModular:THONKICONNNEW
- added R27, R28: 470R, we-rcl:RESISTOR-0805
- added R29, R30, R31, R32, R33, R34, R35, R36, R37: 2.7k, we-rcl:RESISTOR-0805
- 160HZ, 16KHZ, 1KHZ, 2.5KHZ, 410HZ, 63HZ, 7.7KHZ: device MusicThingModular:ALPHA_20MM_ILLUM_FADER -> TomW:ALPHA_20MM_ILLUM_FADER
- R18, R19, R20, R21, R22, R23, R24: value 2k -> 470R
Connections:
- new net N$1: IC6A.OUT, R27.2, R29.1
- new net N$44: R28.1, R_OUT.TIP
- new net N$46: IC6B.OUT, R28.2, R30.1
- new net N$47: IC6B.-IN, R30.2, R32.2, R34.2, R36.2
- new net N$49: IC6A.-IN, R29.2, R31.2, R33.2, R35.2, R37.2
- net +12V: now also IC6P.V+
- net -12V: now also IC6P.V-
- net GND: now also IC6A.+IN, IC6B.+IN, L_OUT.SLEEVE, R_OUT.SLEEVE; no longer IC5A.+IN
- net N$11: no longer C34.1, C35.2
- net N$12: no longer C33.2
- net N$14: no longer C31.1
- net N$18: no longer C31.2
- net N$19: no longer C36.1
- net N$21: now also R33.1
- net N$22: now also L_OUT.TIP, R27.1; no longer IC5A.-IN, IC5A.OUT
- net N$23: no longer C37.1, C38.1
- net N$26: now also R31.1
- net N$27: now also R34.1
- net N$29: now also R32.1
- net N$3: now also IC1A.+IN, R1.1; no longer IC1A.-IN, R2.1
- net N$30: no longer C32.1
- net N$31: no longer C33.1
- net N$33: now also R35.1
- net N$35: now also R36.1
- net N$36: no longer C34.2, C35.1
- net N$37: no longer C36.2
- net N$39: now also R37.1
- net N$4: no longer C32.2
- net N$40: no longer C37.2, C38.2
- net N$7: now also IC1A.-IN, R2.1; no longer IC1A.+IN, R1.1
Other:
- note added: "!"
- note added: "6µF @ 11.5V"
- moved on the sheet: 160HZFADE, 16KHZFADE, 1KHZFADE, 2.5KHZFADE, 410HZFADE, 63HZFADE, 7.7KHZFADE, C10, C11, C14, C15, C16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
