File: graphic_stereo_2.sch (EAGLE design)
At the start: 81 parts, among them IC1 NE5532D, IC2 NE5532D, IC3 NE5532D, IC4 NE5532D, IC5 NE5532D

Commit message: Revert "Tweaks for Rev 1 boards: improve ground plane clearance, move one resistor, move Kills Fascists arwork, small changes to get ground plane to work"
This reverts commit c469b6aed1205b33f2cf1fbab66cd5b8357eaae7.
Parts:
- removed C31, C32, C33, C34, C35, C36, C37, C38: NP, we-rcl:CAPACITOR-0805
- removed OUTPUT: THONKICONNNEW, MusicThingModular:THONKICONNNEW
- added IC6: NE5532D, linear:NE5532D
- added OUTPUTL/MONO, OUTPUT_R: THONKICONNNEW, MusicThingModular:THONKICONNNEW
- added R27, R28: 2.7k, we-rcl:RESISTOR-0805
- added R29, R30: 10k, we-rcl:RESISTOR-0805
- added R31: 470R, we-rcl:RESISTOR-0805
- 160HZ, 16KHZ, 1KHZ, 2.5KHZ, 410HZ, 63HZ, 7.7KHZ: device MusicThingModular:ALPHA_20MM_ILLUM_FADER -> TomW:ALPHA_20MM_ILLUM_FADER
- R18, R19, R20, R21, R22, R23, R24: value 2k -> 470R
Connections:
- new net N$1: 160HZFADE.A, 1KHZFADE.A, 7.7KHZFADE.A, IC6A.+IN, R27.1
- new net N$44: IC6A.OUT, R28.2, R3.2
- new net N$46: 16KHZFADE.E, 2.5KHZFADE.E, 410HZFADE.E, 63HZFADE.E, IC1A.-IN, R2.1
- new net N$47: IC5A.+IN, R29.1, R30.1
- new net N$48: IC5A.-IN, IC5A.OUT, R31.2
- new net N$49: OUTPUTL/MONO.TIP, R31.1
- net GND: now also OUTPUTL/MONO.SLEEVE; no longer IC5A.+IN, OUTPUT.SLEEVE
- net N$11: no longer C34.1, C35.2
- net N$12: no longer C33.2
- net N$14: no longer C31.1
- net N$18: no longer C31.2
- net N$19: no longer C36.1
- net N$22: now also 160HZFADE.E, 1KHZFADE.E, 7.7KHZFADE.E, IC6A.-IN, R28.1; no longer IC5A.-IN, IC5A.OUT
- net N$23: no longer C37.1, C38.1
- net N$3: now also IC1A.+IN, R1.1; no longer 160HZFADE.A, 1KHZFADE.A, 7.7KHZFADE.A, IC1A.-IN, R2.1
- net N$30: no longer C32.1
- net N$31: no longer C33.1
- net N$36: no longer C34.2, C35.1
- net N$37: no longer C36.2
- net N$4: no longer C32.2
- net N$40: no longer C37.2, C38.2
- net N$45: now also R27.2
- net N$5: now also R30.2; no longer R3.2
- net N$6: now also OUTPUT_R.TIP; no longer OUTPUT.TIP
- net N$7: now also OUTPUT_R.SWITCH, R29.2; no longer 160HZFADE.E, 16KHZFADE.E, 1KHZFADE.E, 2.5KHZFADE.E, 410HZFADE.E, 63HZFADE.E, 7.7KHZFADE.E, IC1A.+IN, R1.1
Other:
- note added: "!"
- note added: "6µF @ 11.5V"
- moved on the sheet: C10, C11, C14, C15, C16, C17, C18, C19, C2, C20, C21, C23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
